File: IdcProbe.brd (EAGLE design)
At the start: 50 x 50 mm, 51 parts, among them IC1 TL074D, J2 BNCPTH, X1 MSTBA2, X2 MSTBA2

Commit message: work
Parts:
- removed H1, H2, H3, H4: MOUNT-PAD-ROUND3.2, holes:3,2-PAD
- removed J2: BNCPTH, SparkFun-Connectors:BNC
- added C19, C31, C32: 4.7uF, rcl:C0805
- added C20: 100nF, rcl:C0805
- added C21: 6.8pF, rcl:C0805
- added C22, C23, C28, C29, C33, C34, C35, C36: 10uF, rcl:C1206
- added C25: 10nF, rcl:C0805
- added C26: 4.7nF, rcl:C0805
- added C27: 220nF, rcl:C0805
- added C30: 7.5pF, rcl:C0805
- added CN1: (no value), microbuilder:USB-MINIB_LARGER
- added D2, D3, D4: MBR0520, diode:SOD123
- added L1, L2: 3.3uH, Jeroen:VLS3015
- added L3, L4: extra 3.3uH, Jeroen:VLS3015
- added LD1, LD2, LD3: (no value), led:CHIP-LED0805
- added P1, P2: BANANA_SOCKETVERTICAL, Jeroen:4,5-PAD
- added R12, R2: 10k, rcl:R0805I
- added R13: 100, rcl:R0805I
- added R14, R17: 1000k, rcl:R0805I
- added R15, R16: 100k, rcl:R0805I
- added R18, R19: 3.9k, rcl:R0805I
- added R20: 1.5k, rcl:R0805I
- added TP1: V+, Jeroen:TESTHOOK
- added TP10, TP12, TP2, TP3, TP7: TESTPOINT_GND, Jeroen:PROBE_POINT
- added U$1: PCB_HAMMOND_1591XXL, Jeroen:HMD_MFG_1591XXL
- added U2: TPS65131RGET, Jeroen:QFN50P400X400X100-25N
- added X3: R141426, con-coax:R141426
- added X4: MSTBA2, con-phoenix-508:MSTBA2
- PS1: device Jeroen:SIP-7_RP -> Jeroen:SIP-7_RD
- moved C1 64.0 mm to (106.6, 22.4)
- moved C10 64.0 mm to (86.9, 15.8)
- moved C11 64.0 mm to (75.0, 37.1)
- moved C12 64.0 mm to (75.0, 34.6)
- moved C2 64.0 mm to (107.9, 24.9)
- moved C24 64.0 mm to (95.8, 35.2)
- moved C3 64.0 mm to (106.6, 19.9)
- moved C5 64.0 mm to (95.8, 37.6)
- moved C6 64.0 mm to (102.8, 19.9)
- moved C7 64.0 mm to (101.5, 24.9)
- moved C8 64.0 mm to (102.8, 22.4)
- moved C9 64.0 mm to (103.4, 11.6)
- moved D1 64.0 mm to (101.5, 36.4)
- moved R1 64.0 mm to (106.6, 17.3)
- moved R10 64.0 mm to (102.8, 17.3)
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Connections:
- new net CN: C26.1, U2.18
- new net CP: C25.1, U2.21
- new net FBN: C30.1, R16.1, R17.1, U2.16
- new net FBP: C21.2, R14.1, R15.2, U2.22
- new net INP: D2.A, L1.2, U2.1, U2.24
- new net N$12: LD3.A, R19.2
- new net N$13: IC1.2, R12.2, R2.1
- new net N$14: CN1.VBUS, D4.A, X4.1
- new net N$15: LD1.A, R20.1
- new net N$4: LD2.A, R18.1
- new net OUTN: D3.C, L2.2, U2.13, U2.14
- new net RV+: C21.1, C22.1, C33.1, D2.C, L4.1, R14.2, TP2.TP, U2.23
- new net RV-: C23.1, C30.2, C35.1, D3.A, L3.1, R17.2, TP12.TP, U2.15
- new net VI: C19.1, C31.1, C32.1, D4.C, L1.1, R13.2, R20.2, TP7.TP, U2.5, U2.6
- new net VIN1: C20.1, R13.1, U2.10, U2.11, U2.4, U2.8, U2.9
- new net VREF: C27.1, R16.2, U2.17
- net +15V: now also PS1.6; no longer PS1.7
- net -15V: now also PS1.4; no longer PS1.5
- net GND: now also C14.+, C19.2, C20.2, C22.2, C23.2, C25.2, C26.2, C27.2, C28.2, C29.2, C31.2, C32.2, C33.2, C34.2, C35.2, C36.2, CN1.GND, L2.1, LD1.C, LD2.C, LD3.C, PS1.5, R12.1, R15.1, TP1.TP, TP10.GND, TP12.GND, TP2.GND, TP3.GND, TP7.GND, U2.19, U2.2, U2.25, U2.3, X3.2, X3.3, X3.4, X3.5, X4.2; no longer C14.-, J2.GND, PS1.6
- net N$1: now also X3.1; no longer J2.S
- net N$2: now also P1.B4,5
- net N$3: now also P2.B4,5
- net N$9: now also R2.2; no longer IC1.2
- net V+: now also C29.1, C34.1, L4.2, R18.2, TP3.TP
- net V-: now also C14.-, C28.1, C36.1, L3.2, R19.1, TP10.TP; no longer C14.+
Routing:
- net V+: track 113.8 -> 0.00 mm, vias 3 -> 0
- net V-: track 107.4 -> 0.00 mm, vias 3 -> 0
- net GND: track 55.5 -> 17.8 mm, vias 6 -> 2
- net -15V: track 29.1 -> 0.00 mm
- net N$10: track 18.7 -> 39.5 mm
- net +15V: track 18.1 -> 0.00 mm
- net PWR_VIN: track 17.0 -> 0.00 mm
- net PGND: track 9.26 -> 0.00 mm
- net N$42: track 7.63 -> 0.00 mm
- net N$40: track 7.63 -> 0.00 mm
- net N$13: track 0.00 -> 6.47 mm
- net N$38: track 5.92 -> 0.00 mm
- net N$6: track 5.85 -> 0.00 mm
- net N$5: track 5.52 -> 0.00 mm
- net N$11: track 5.36 -> 0.00 mm
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- added copper zone on layer 1, net N$2
- added copper zone on layer 1, net N$3
Other:
- board size 50 x 50 mm -> 50 x 80 mm
- board text added: "5A max"
- board text added: "5A/5V"
- board text added: "IdcProbe"
- board text added: "IdcProbe 5A max"
- board text added: "Jeroen Lodder 2017-09"
- board text added: "Vin 12V Vout 5A/5V"

Commit message: update
Parts:
- removed C27: 220nF, rcl:C0805
- removed C28, C29, C33, C34, C35, C36: 10uF, rcl:C1206
- removed C30: 7.5pF, rcl:C0805
- removed C31, C32: 4.7uF, rcl:C0805
- removed CN1: (no value), microbuilder:USB-MINIB_LARGER
- removed D1: SS24A, diode:DO-214AC
- removed D4: MBR0520, diode:SOD123
- removed LD1: (no value), led:CHIP-LED0805
- removed PS1: RP-1215D, Jeroen:SIP-7_RD
- removed R1: 240, rcl:R0805
- removed R15, R16: 100k, rcl:R0805I
- removed R17: 1000k, rcl:R0805I
- removed R18, R19: 3.9k, rcl:R0805I
- removed R20: 1.5k, rcl:R0805I
- removed TP10, TP12, TP3: TESTPOINT_GND, Jeroen:PROBE_POINT
- removed TP11, TP15, TP6: GND, Jeroen:TESTHOOK
- removed TP13: +15V, Jeroen:TESTHOOK
- removed TP14: V+, Jeroen:TESTHOOK
- removed VREG1: VREG_3PINS_ADJ-LM317T-TO-220VA, dp_devices:TO-220V
- removed VREG2: VREG_3PINS_ADJ-LM337T-TO-220VB, dp_devices:TO-220V
- removed X1, X2, X4: MSTBA2, con-phoenix-508:MSTBA2
- added J1: (no value), SparkFun-Connectors:MOLEX-1X2
- C1, C3: value 100nF -> 4.7uF
- C10: value 100nF -> 6.8pF
- C11, C12: value 100nF -> 10uF; device rcl:C0805 -> rcl:C1206
- C13, C14: value 47uF -> 10uF; device rcl:PANASONIC_D -> rcl:C1206
- C15: value 3.3nF -> 10uF; device rcl:C0805 -> rcl:C1206
- C16, C17: value (none) -> 10uF; device rcl:C0805 -> rcl:C1206
- C18: value (none) -> 100nF
- C19: value 4.7uF -> 100nF
- C2: value 10uF -> 4.7uF; device rcl:C1206 -> rcl:C0805
- C21: value 6.8pF -> 47uF; device rcl:C0805 -> rcl:PANASONIC_D
- C22: value 10uF -> 47uF; device rcl:C1206 -> rcl:PANASONIC_D
- C23: value 10uF -> 3.3nF; device rcl:C1206 -> rcl:C0805
- C24: value 100nF -> (none)
- C25: value 10nF -> (none)
- C26: value 4.7nF -> (none)
- C4: value 2.2uF -> 100nF
- C5: value 1uF -> 10nF
- C6: value 100nF -> 4.7nF
- C7: value 10uF -> 220nF; device rcl:C1206 -> rcl:C0805
- C8: value 100nF -> 7.5pF
- C9: value 2.2uF -> 10uF; device rcl:C0805 -> rcl:C1206
- R10: value 240 -> (none)
- R11: value 10k -> (none)
- R12: device rcl:R0805I -> rcl:R0805
- R13: value 100 -> 10k
- R14: value 1000k -> 10k
- R2: value 10k -> 100
- R3, R6: value 2.2k -> 100k; device rcl:R0805 -> rcl:R0805I
- R4: value (none) -> 1000k; device rcl:R0805 -> rcl:R0805I
- R5: value 15 -> 1000k; device rcl:R0805 -> rcl:R0805I
- R7: value (none) -> 3.9k; device rcl:R0805 -> rcl:R0805I
- R8: value 33k -> 3.9k; device rcl:R0805 -> rcl:R0805I
- R9: value 33k -> 15
- TP1, TP4: value V+ -> (none)
- TP5: value GND -> TESTPOINT_GND; device Jeroen:TESTHOOK -> Jeroen:PROBE_POINT
- TP8: value V- -> (none)
- TP9: value -15V -> TESTPOINT_GND; device Jeroen:TESTHOOK -> Jeroen:PROBE_POINT
- U1: value (none) -> TPS65131RGET; device Jeroen:CMS3005 -> Jeroen:QFN50P400X400X100-25N
- U2: value TPS65131RGET -> (none); device Jeroen:QFN50P400X400X100-25N -> Jeroen:CMS3005
- moved D3 128.6 mm to (17.5, 53.0), turned to 270 degrees
- moved D2 117.0 mm to (5.50, 48.0)
- moved C26 115.7 mm to (34.0, 56.0), turned to 270 degrees
- moved R13 112.3 mm to (32.0, 50.0), turned to 90 degrees
- moved R3 108.4 mm to (11.5, 58.0), turned to 270 degrees
- moved C25 106.0 mm to (28.2, 38.2)
- moved C6 103.2 mm to (6.50, 57.0), turned to 180 degrees
- moved LD2 101.9 mm to (46.0, 25.0), turned to 270 degrees
- moved C23 100.5 mm to (28.2, 40.5)
- moved C2 99.0 mm to (10.5, 43.0), turned to 90 degrees
- moved C4 98.9 mm to (12.5, 44.0), turned to 270 degrees
- moved R6 98.9 mm to (7.50, 51.0), turned to 90 degrees
- moved C3 98.7 mm to (9.50, 37.5)
- moved C1 98.6 mm to (9.50, 39.5)
- moved LD3 98.5 mm to (46.0, 22.5), turned to 270 degrees
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Connections:
- removed net +15V: C1.2, C2.2, PS1.6, TP13.TP, VREG1.3
- removed net -15V: C6.1, C7.1, PS1.4, TP9.TP, VREG2.2
- removed net N$15 (its old number): LD1.A, R20.1
- removed net N$3: P2.B4,5, U1.7, X2.1
- removed net N$38: D1.A, X1.1
- removed net N$4: LD2.A, R18.1
- removed net N$40: R1.2, R3.2, R8.2, VREG1.1
- removed net N$42: R10.2, R6.1, R9.1, VREG2.1
- removed net N$7 (its old number): C15.2, R5.2
- removed net N$8 (its old number): C17.2, R4.2
- removed net PGND: C24.2, C5.2, PS1.2, X1.2
- removed net PWR_VIN: C24.1, C5.1, D1.C, PS1.1
- removed net VIN1: C20.1, R13.1, U2.10, U2.11, U2.4, U2.8, U2.9
- new net N$11: IC1.1, R11.1, R12.2, R13.2
- new net N$5: P1.B4,5, U2.6
- new net N$6: P2.B4,5, U2.7
- new net VIN: C4.1, R2.1, U1.10, U1.11, U1.4, U1.8, U1.9
- net CN: now also C6.1, U1.18; no longer C26.1, U2.18
- net CP: now also C5.1, U1.21; no longer C25.1, U2.21
- net FBN: now also C8.1, R3.1, R4.1, U1.16; no longer C30.1, R16.1, R17.1, U2.16
- net FBP: now also C10.2, R5.1, R6.2, U1.22; no longer C21.2, R14.1, R15.2, U2.22
- net GND: now also C1.2, C11.2, C12.2, C13.2, C14.2, C15.2, C16.2, C17.2, C19.1, C2.2, C20.1, C21.-, C22.+, C23.1, C24.1, C25.1, C26.1, C3.2, C4.2, C5.2, J1.1, R14.1, R6.1, TP5.GND, TP8.TP, TP9.GND, U1.19, U1.2, U1.25, U2.4; no longer C1.1, C11.1, C12.1, C13.-, C14.+, C15.1, C16.1, C17.1, C18.1, C19.2, C2.1, C20.2, C22.2, C23.2, C25.2, C26.2, C27.2, C28.2, C29.2, C3.1, C31.2, C32.2, C33.2, C34.2, C35.2, C36.2, C4.1, C8.2, CN1.GND, LD1.C, PS1.5, R11.1, R15.1, R3.1, R6.2, R8.1, R9.2, TP10.GND, TP11.TP, TP12.GND, TP15.TP, TP3.GND, TP6.TP, U1.4, U2.19, U2.2, U2.25, X4.2
- net INP: now also U1.1, U1.24; no longer U2.1, U2.24
- net N$1: now also LD2.A, R7.1; no longer C18.2, R7.2, TP5.TP, X3.1
- net N$10: now also C25.2, R10.2; no longer C16.2, IC1.3, R4.1, R5.1, U1.5
- net N$12: now also C26.2, R11.2, TP9.TP, X3.1; no longer LD3.A, R19.2
- net N$13: now also C24.2, IC1.3, R10.1, R9.1, TP7.TP, U2.5; no longer IC1.2, R12.2, R2.1
- net N$14: now also IC1.2, R13.1, R14.2; no longer CN1.VBUS, D4.A, X4.1
- net N$2: now also LD3.A, R8.2; no longer P1.B4,5, U1.6, X2.2
- net N$9: now also C23.2, R9.2; no longer IC1.1, R11.2, R2.2, R7.1
- net OUTN: now also U1.13, U1.14; no longer U2.13, U2.14
- net RV+: now also C10.1, C11.1, C14.1, R5.2, U1.23; no longer C21.1, C22.1, C33.1, R14.2, TP2.TP, U2.23
- net RV-: now also C16.1, C8.2, C9.1, R4.2, U1.15; no longer C23.1, C30.2, C35.1, R17.2, TP12.TP, U2.15
- net V+: now also C13.1, C15.1, C18.2, C19.2, C21.+, R7.2, TP2.TP, U2.1; no longer C10.2, C11.2, C13.+, C29.1, C3.2, C34.1, C4.2, R1.1, R18.2, TP14.TP, TP3.TP, U1.1, VREG1.2
- net V-: now also C12.1, C17.1, C18.1, C20.2, C22.-, R8.1, TP5.TP, U2.2; no longer C10.1, C12.2, C14.-, C28.1, C36.1, C8.1, C9.1, R10.1, R19.1, TP10.TP, TP8.TP, U1.2, VREG2.3
- net VI: now also C1.1, C2.1, C3.1, J1.2, R2.2, U1.5, U1.6; no longer C19.1, C31.1, C32.1, D4.C, R13.2, R20.2, TP7.TP, U2.5, U2.6
- net VREF: now also C7.1, R3.2, U1.17; no longer C27.1, R16.2, U2.17
Routing:
- net GND: track 17.8 -> 120.6 mm, vias 2 -> 18
- net V+: track 0.00 -> 74.6 mm, vias 0 -> 2
- net V-: track 0.00 -> 70.2 mm, vias 0 -> 4
- net N$10: track 39.5 -> 2.35 mm
- net N$13: track 6.47 -> 34.0 mm
- net RV-: track 0.00 -> 20.5 mm, vias 0 -> 2
- net N$12: track 0.00 -> 20.4 mm
- net VIN: track 0.00 -> 19.2 mm, vias 0 -> 2
- net RV+: track 0.00 -> 17.5 mm
- net N$1: track 14.0 -> 2.90 mm
- net N$11: track 0.00 -> 11.0 mm
- net FBN: track 0.00 -> 9.61 mm
- net VI: track 0.00 -> 8.62 mm, vias 0 -> 1
- net N$14: track 0.00 -> 7.54 mm
- net FBP: track 0.00 -> 7.21 mm
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- added copper zone on layer 1, net INP
- added copper zone on layer 1, net N$5
- added copper zone on layer 16, net N$5
- added copper zone on layer 1, net N$6
- added copper zone on layer 16, net N$6
- added copper zone on layer 1, net OUTN
- added copper zone on layer 1, net VI
- removed copper zone on layer 1, net N$2
- removed copper zone on layer 16, net N$2
- removed copper zone on layer 1, net N$3
- removed copper zone on layer 16, net N$3
Other:
- board text added: "Prototype TPS65131 Jeroen Lodder 10-2017"
- board text added: "V+"
- board text added: "V-"
- board text removed: "5A max"
- board text removed: "5A/5V"
- board text removed: "IdcProbe"
- board text removed: "IdcProbe 5A max"
- board text removed: "Jeroen Lodder 2017-09"
- board text removed: "Vin 12V Vout 5A/5V"

Commit message: work
Parts:
- removed C15, C17: 10uF, rcl:C1206
- removed U2: (no value), Jeroen:CMS3005
- added D6: SS24 (40V), microbuilder:SMADIODE
- added LED1: (no value), led:LED3MM
- added R1: 1K, rcl:R0805
- added R15: 2M, rcl:R0805
- added R16: 100k, Jeroen:3386-MULTI
- added R17: 100, rcl:R0805I
- added U3: (no value), Jeroen:CMS3015
- R11: value (none) -> 0
- R12: value 10k -> 100k
- moved TP8 19.0 mm to (46.5, 58.5)
- moved TP7 17.1 mm to (31.5, 43.5), turned to 0 degrees
- moved C25 12.8 mm to (28.0, 51.0), turned to 270 degrees
- moved C24 11.5 mm to (32.0, 47.0), turned to 270 degrees
- moved C23 10.6 mm to (30.0, 51.0), turned to 270 degrees
- moved R10 9.84 mm to (28.0, 47.0), turned to 90 degrees
- moved R9 6.96 mm to (30.0, 47.0), turned to 90 degrees
- moved R14 4.47 mm to (34.0, 50.0), turned to 270 degrees
- moved TP2 4.12 mm to (4.50, 34.5)
- moved R13 4.00 mm to (36.0, 50.0)
- moved C21 3.16 mm to (5.00, 25.0)
- moved J1 2.75 mm to (10.0, 31.0), flipped to the bottom, turned to 0 degrees
- moved TP5 2.46 mm to (16.8, 37.0), turned to 180 degrees
- moved C22 2.24 mm to (17.0, 25.0)
- moved C18 2.00 mm to (42.0, 41.0)
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Connections:
- new net N$16: LED1.A, R17.1
- new net N$3: IC1.3, IC1.7, R1.2
- new net N$4: IC1.6, R1.1, R15.2
- net GND: now also D6.A, LED1.K, U3.3, U3.4; no longer C15.2, C17.2, IC1.5, U2.3, U2.4
- net N$13: now also IC1.5, U3.5; no longer IC1.3, U2.5
- net N$15: now also R15.1, R16.2, R16.5, R16.7; no longer IC1.6, IC1.7
- net N$5: now also U3.6, U3.6'; no longer U2.6
- net N$6: now also U3.7, U3.7'; no longer U2.7
- net V+: now also R16.3, R16.6, R17.2, U3.1; no longer C15.1, U2.1
- net V-: now also R16.1, R16.4, U3.2; no longer C17.1, U2.2
- net VI: now also D6.C
Routing:
- net GND: track 120.6 -> 85.8 mm, vias 18 -> 27
- net V-: track 70.2 -> 88.5 mm
- net V+: track 74.6 -> 86.9 mm
- net N$3: track 0.00 -> 11.5 mm, vias 0 -> 2
- net N$4: track 0.00 -> 5.62 mm
- net N$13: track 34.0 -> 39.2 mm
- net N$15: track 4.19 -> 7.59 mm
- net VI: track 8.62 -> 12.0 mm
- net N$16: track 0.00 -> 3.09 mm
- net N$14: track 7.54 -> 5.64 mm
- net N$11: track 11.0 -> 12.3 mm
- net N$2: vias 0 -> 1
- net N$1: vias 0 -> 1
Other:
- board text added: "- +"
- board text added: "5A (pulsed 20A) 1A/V 2MHz"
- board text added: "5V input"
- board text added: "Idc probe V1"
- board text added: "Iin"
- board text added: "Iout"
- board text added: "No magnetic tools!"
- board text added: "Offset"
- board text removed: "Prototype TPS65131 Jeroen Lodder 10-2017"

Commit message: Ordered
Parts:
- moved C22 16.0 mm to (33.0, 25.0), flipped to the bottom
- moved C21 12.0 mm to (17.0, 25.0), flipped to the bottom
- moved TP8 2.00 mm to (46.5, 60.5)
Routing:
- net V+: track 86.9 -> 97.3 mm
- net V-: track 88.5 -> 87.8 mm
- net GND: vias 27 -> 37
Other:
- board text added: "5A/15A (pulsed 20A/60A) CMS3005 / CMS3015"
- board text added: "Idc Probe V1"
- board text added: "Jeroen Lodder 2017-10"
- board text removed: "5A (pulsed 20A) 1A/V 2MHz"
- board text removed: "Idc probe V1"
- board text removed: "No magnetic tools!"

Commit message: added notes, fixed some values
Parts:
- R14: value 10k -> (none)
- R15: value 2M -> 1.8M
- R17: value 100 -> 3.9k
Other:
- board text added: "Need to fix layout: - No 1206 but 0806 capacitors - Lower ground impedance, more vias. - Make sure control TPS signals are cuttable on other layer. - Mount holes slightly large"
Changed lines of the file:
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@@
 CMS3005 / CMS3015</text>
 <text x="25" y="45.75" size="1.27" layer="22" ratio="15" rot="MR0" align="bottom-center">Jeroen Lodder 2017-10</text>
+<text x="91" y="-5" size="1.778" layer="19" rot="R180">Need to fix layout:
+- No 1206 but 0806 capacitors
+- Lower ground impedance, more vias.
+- Make sure control TPS signals are cuttable on other layer.
+- Mount holes slightly large</text>
 </plain>
 <attributes>
@@
 <attribute name="VALUE" x="38.54" y="49.365" size="0.8" layer="27" ratio="15" rot="R90"/>
 </element>
-<element name="R14" library="rcl" package="R0805I" value="10k" x="34" y="50" smashed="yes" rot="R270">
+<element name="R14" library="rcl" package="R0805I" value="" x="34" y="50" smashed="yes" rot="R270">
 <attribute name="NAME" x="34.48" y="45.865" size="0.8" layer="25" ratio="15" rot="R90"/>
 <attribute name="VALUE" x="31.46" y="50.635" size="0.8" layer="27" ratio="15" rot="R270"/>
@@
 <attribute name="VALUE" x="33.46" y="43.635" size="0.8" layer="27" ratio="15" rot="R270"/>
 </element>
-<element name="R15" library="rcl" package="R0805" value="2M" x="34" y="43" smashed="yes" rot="R90">
+<element name="R15" library="rcl" package="R0805" value="1.8M" x="34" y="43" smashed="yes" rot="R90">
 <attribute name="NAME" x="32.635" y="41.73" size="0.8" layer="25" ratio="15" rot="R180"/>
 <attribute name="VALUE" x="36.54" y="42.365" size="0.8" layer="27" ratio="15" rot="R90"/>
@@
 <attribute name="VALUE" x="26.905" y="38.349" size="1.27" layer="27" ratio="10"/>
 </element>
-<element name="R17" library="rcl" package="R0805I" value="100" x="25" y="37" smashed="yes">
+<element name="R17" library="rcl" package="R0805I" value="3.9k" x="25" y="37" smashed="yes">
 <attribute name="NAME" x="27.365" y="36.27" size="0.8" layer="25" ratio="15"/>
 <attribute name="VALUE" x="24.365" y="34.46" size="0.8" layer="27" ratio="15"/>
