File: IdcProbe.brd (EAGLE design)
At the start: 50 x 80 mm, 79 parts, among them IC1 TL074D, P1 BANANA_SOCKETVERTICAL, P2 BANANA_SOCKETVERTICAL, Q1 PMV45EN, U1 NCP361MUTBG, U2 TPS65131RGET, X1 R141426

Commit message: ordered rev2
Parts:
- C10: value 220nF -> 220nF 25V X7R
- C26: value 3.3nF / 2.2nF -> 3.3nF / 2.2nF 25V NP0
- F1: value 0.5AT -> 1AF; device dp_devices:PTC0805 -> Jeroen:1206_HV
- J1: value (none) -> PSL2G
- R18: value (none) -> open/15K
- R19: value (none) -> 10k/open
- U3: value (none) -> CMS3005
- moved LED1 10.0 mm to (25.0, 50.0), turned to 180 degrees
- moved R7 3.00 mm to (25.0, 40.0), turned to 270 degrees
- moved C30 1.00 mm to (42.0, 40.0)
- moved F1 0.50 mm to (15.0, 26.0)
- moved Q1 0.50 mm to (15.0, 31.5)
Connections:
- net N$18: now also F1.P$1; no longer F1.1
- net N$21: now also F1.P$2; no longer F1.2
Routing:
- net N$16: track 3.09 -> 9.48 mm
- net V+: track 90.9 -> 93.7 mm
- net N$18: track 7.31 -> 6.40 mm
- net N$19: track 5.07 -> 5.57 mm
- net GND: vias 96 -> 95

Commit message: Accumulated fixes during testing for version 1.2
Parts:
- R22: value 0 -> 270
- moved R22 6.08 mm to (38.0, 53.0)
- moved TP9 3.58 mm to (38.0, 58.2)
- moved C31 2.24 mm to (32.0, 55.0)
- moved R21 1.00 mm to (30.0, 55.0)
Connections:
- removed net N$12: C31.2, R22.2, TP9.TP, X1.1
- new net N$22: IC1.1, R22.1
- net N$11: now also C31.2, R22.2, TP9.TP, X1.1; no longer IC1.1, R22.1
Routing:
- net N$12: track 20.4 -> 0.00 mm
- net N$11: track 12.6 -> 28.8 mm
- net GND: track 104.4 -> 99.9 mm, vias 95 -> 120
- net N$22: track 0.00 -> 3.53 mm
