File: IdcProbe.sch (EAGLE design)
At the start: 79 parts, among them IC1 TL074D, P1 BANANA_SOCKETVERTICAL, P2 BANANA_SOCKETVERTICAL, Q1 PMV45EN, U1 NCP361MUTBG, U2 TPS65131RGET, X1 R141426

Commit message: ordered rev2
Parts:
- C10: value 220nF -> 220nF 25V X7R
- C26: value 3.3nF / 2.2nF -> 3.3nF / 2.2nF 25V NP0
- F1: value 0.5AT -> 1AF; device dp_devices:FUSE_PTC-0805 -> Jeroen:FUSE1206
- J1: value (none) -> PSL2G; MPN TMK212AB7475KG-T -> (none)
- R18: value (none) -> open/15K
- R19: value (none) -> 10k/open
- U3: value (none) -> CMS3005
Connections:
- net N$18: now also F1.P$1; no longer F1.1
- net N$21: now also F1.P$2; no longer F1.2
Other:
- note added: "Overcurrent protection U1 (F1)"
- note added: "Overvoltage protection U1"
- note added: "Transient protection D1"
- note removed: "Overcurrent protection U2"
- note removed: "Overvoltage protection U2"
- note removed: "Transient protection D5"

Commit message: Accumulated fixes during testing for version 1.2
Parts:
- R22: value 0 -> 270
Connections:
- removed net N$12: C31.2, R22.2, TP9.P$1, X1.1
- new net N$22: IC1A.OUT, R22.1
- net N$11: now also C31.2, R22.2, TP9.P$1, X1.1; no longer IC1A.OUT, R22.1
Other:
- moved on the sheet: C31, R20, R21, R22, TP9
